File: mcp2515.sch (KiCad schematic (older format))
At the start: 14 parts, among them J3 Conn_01x02, J4 Conn_01x06, U1 TJA1051T, U2 MCP2515-xSO, X1 Crystal

Commit message: Added  Values for Capacitors, added Footprints
Parts:
- added JP?: SolderJumper_2_Open, symbol Jumper:SolderJumper_2_Open
- C1: value CP -> 10uF/16V
- C2, C5: value C -> 0,1uF; footprint (none) -> Capacitor_SMD:C_0201_0603Metric
- C3: value C -> 22pF; footprint (none) -> Capacitor_SMD:C_0201_0603Metric
- C4: renamed from C?; value C -> 22pF; footprint (none) -> Capacitor_SMD:C_0201_0603Metric
- POW: footprint (none) -> LED_SMD:LED_0603_1608Metric
- R1, R2: footprint (none) -> Resistor_SMD:R_0603_1608Metric
- R3: value 10k07 -> 10k; footprint (none) -> Resistor_SMD:R_0603_1608Metric
- X1: value Crystal -> C115962; footprint (none) -> Crystal:Crystal_SMD_5032-2Pin_5.0x3.2mm
Connections:
- net at J3.1 (Pin_1), U1.7 (CANH): now also R2.2; no longer R2.1
- net at J3.2 (Pin_2), U1.6 (CANL): now also JP?.2 (B); no longer R2.2
- new net: JP?.1 (A), R2.1
Other:
- moved on the sheet: C1, C2, C5, J3, POW, R1, R2
Changed lines of the file:
@@
 EESchema Schematic File Version 4
+LIBS:mcp2515-cache
 EELAYER 30 0
 EELAYER END
@@
 Wire Wire Line
 	4000 3700 4300 3700
-Connection ~ 7150 4850
-Wire Wire Line
-	7150 4850 7450 4850
-Connection ~ 7150 4550
 $Comp
 L Device:R R1
 U 1 1 5E9187AF
-P 7300 4550
-F 0 "R1" V 7093 4550 50  0000 C CNN
-F 1 "1k" V 7184 4550 50  0000 C CNN
-F 2 "" V 7230 4550 50  0001 C CNN
-F 3 "~" H 7300 4550 50  0001 C CNN
-	1    7300 4550
-	0    1    1    0
-$EndComp
-Wire Wire Line
-	6950 4850 7150 4850
-Connection ~ 6950 4850
+P 7700 4550
+F 0 "R1" V 7493 4550 50  0000 C CNN
+F 1 "1k" V 7584 4550 50  0000 C CNN
+F 2 "Resistor_SMD:R_0603_1608Metric" V 7630 4550 50  0001 C CNN
+F 3 "~" H 7700 4550 50  0001 C CNN
+	1    7700 4550
+	0    1    1    0
+$EndComp
 $Comp
 L power:GND #PWR?
 U 1 1 5E916F4B
-P 6950 4850
-F 0 "#PWR?" H 6950 4600 50  0001 C CNN
-F 1 "GND" H 6955 4677 50  0000 C CNN
-F 2 "" H 6950 4850 50  0001 C CNN
-F 3 "" H 6950 4850 50  0001 C CNN
-	1    6950 4850
-	1    0    0    -1
-$EndComp
-Wire Wire Line
-	6950 4550 7150 4550
-Connection ~ 6950 4550
-Wire Wire Line
-	6800 4850 6950 4850
-Connection ~ 6800 4850
-Wire Wire Line
-	6400 4850 6800 4850
-Wire Wire Line
-	6800 4550 6950 4550
-Connection ~ 6800 4550
-Wire Wire Line
-	6400 4550 6800 4550
+P 7150 4850
+F 0 "#PWR?" H 7150 4600 50  0001 C CNN
+F 1 "GND" H 7155 4677 50  0000 C CNN
+F 2 "" H 7150 4850 50  0001 C CNN
+F 3 "" H 7150 4850 50  0001 C CNN
+	1    7150 4850
+	1    0    0    -1
+$EndComp
 $Comp
 L Device:LED POW
 U 1 1 5E91395F
-P 7450 4700
-F 0 "POW" V 7489 4583 50  0000 R CNN
-F 1 "LED" V 7398 4583 50  0000 R CNN
-F 2 "" H 7450 4700 50  0001 C CNN
-F 3 "~" H 7450 4700 50  0001 C CNN
-	1    7450 4700
+P 7850 4700
+F 0 "POW" V 7889 4583 50  0000 R CNN
+F 1 "LED" V 7798 4583 50  0000 R CNN
+F 2 "LED_SMD:LED_0603_1608Metric" H 7850 4700 50  0001 C CNN
+F 3 "~" H 7850 4700 50  0001 C CNN
+	1    7850 4700
 	0    -1   -1   0
 $EndComp
@@
 L Device:C C5
 U 1 1 5E913314
-P 7150 4700
-F 0 "C5" H 7265 4746 50  0000 L CNN
-F 1 "C" H 7265 4655 50  0000 L CNN
-F 2 "" H 7188 4550 50  0001 C CNN
-F 3 "~" H 7150 4700 50  0001 C CNN
-	1    7150 4700
+P 7350 4700
+F 0 "C5" H 7465 4746 50  0000 L CNN
+F 1 "0,1uF" H 7465 4655 50  0000 L CNN
+F 2 "Capacitor_SMD:C_0201_0603Metric" H 7388 4550 50  0001 C CNN
+F 3 "~" H 7350 4700 50  0001 C CNN
+	1    7350 4700
 	1    0    0    -1
 $EndComp
@@
 L Device:C C2
 U 1 1 5E912C6B
-P 6800 4700
-F 0 "C2" H 6915 4746 50  0000 L CNN
-F 1 "C" H 6915 4655 50  0000 L CNN
-F 2 "" H 6838 4550 50  0001 C CNN
-F 3 "~" H 6800 4700 50  0001 C CNN
-	1    6800 4700
+P 6900 4700
+F 0 "C2" H 7015 4746 50  0000 L CNN
+F 1 "0,1uF" H 7015 4655 50  0000 L CNN
+F 2 "Capacitor_SMD:C_0201_0603Metric" H 6938 4550 50  0001 C CNN
+F 3 "~" H 6900 4700 50  0001 C CNN
+	1    6900 4700
 	1    0    0    -1
 $EndComp
@@
 L Device:CP C1
 U 1 1 5E9123FE
-P 6400 4700
-F 0 "C1" H 6518 4746 50  0000 L CNN
-F 1 "CP" H 6518 4655 50  0000 L CNN
-F 2 "" H 6438 4550 50  0001 C CNN
-F 3 "~" H 6400 4700 50  0001 C CNN
-	1    6400 4700
+P 6250 4700
+F 0 "C1" H 6368 4746 50  0000 L CNN
+F 1 "10uF/16V" H 6368 4655 50  0000 L CNN
+F 2 "" H 6288 4550 50  0001 C CNN
+F 3 "~" H 6250 4700 50  0001 C CNN
+	1    6250 4700
 	1    0    0    -1
 $EndComp
@@
 L power:VCC #PWR?
 U 1 1 5E911F3B
-P 6950 4550
-F 0 "#PWR?" H 6950 4400 50  0001 C CNN
-F 1 "VCC" H 6967 4723 50  0000 C CNN
-F 2 "" H 6950 4550 50  0001 C CNN
-F 3 "" H 6950 4550 50  0001 C CNN
-	1    6950 4550
+P 7000 4550
+F 0 "#PWR?" H 7000 4400 50  0001 C CNN
+F 1 "VCC" H 7017 4723 50  0000 C CNN
+F 2 "" H 7000 4550 50  0001 C CNN
+F 3 "" H 7000 4550 50  0001 C CNN
+	1    7000 4550
 	1    0    0    -1
 $EndComp
@@
 P 5800 4650
 F 0 "R3" H 5870 4696 50  0000 L CNN
-F 1 "10k07" H 5870 4605 50  0000 L CNN
-F 2 "" V 5730 4650 50  0001 C CNN
+F 1 "10k" H 5870 4605 50  0000 L CNN
+F 2 "Resistor_SMD:R_0603_1608Metric" V 5730 4650 50  0001 C CNN
 F 3 "~" H 5800 4650 50  0001 C CNN
 	1    5800 4650
@@
 $EndComp
 Wire Wire Line
-	7300 3900 7600 3900
-Connection ~ 7300 3900
-Wire Wire Line
-	7600 3900 7600 3700
-Wire Wire Line
-	7100 3900 7300 3900
-Wire Wire Line
-	7300 3600 7600 3600
-Connection ~ 7300 3600
-Wire Wire Line
-	7150 3600 7300 3600
-Wire Wire Line
-	7150 3700 7150 3600
-Wire Wire Line
 	7100 3700 7150 3700
 $Comp
@@
 	4150 4300 4000 4300
 $Comp
-L Device:C C?
+L Device:C C4
 U 1 1 5E8FD77A
 P 3700 4600
-F 0 "C?" V 3448 4600 50  0000 C CNN
-F 1 "C" V 3539 4600 50  0000 C CNN
-F 2 "" H 3738 4450 50  0001 C CNN
+F 0 "C4" V 3448 4600 50  0000 C CNN
+F 1 "22pF" V 3539 4600 50  0000 C CNN
+F 2 "Capacitor_SMD:C_0201_0603Metric" H 3738 4450 50  0001 C CNN
 F 3 "~" H 3700 4600 50  0001 C CNN
 	1    3700 4600
@@
 P 3850 4300
 F 0 "C3" V 3598 4300 50  0000 C CNN
-F 1 "C" V 3689 4300 50  0000 C CNN
-F 2 "" H 3888 4150 50  0001 C CNN
+F 1 "22pF" V 3689 4300 50  0000 C CNN
+F 2 "Capacitor_SMD:C_0201_0603Metric" H 3888 4150 50  0001 C CNN
 F 3 "~" H 3850 4300 50  0001 C CNN
 	1    3850 4300
@@
 L Device:R R2
 U 1 1 5E8FF39E
-P 7300 3750
-F 0 "R2" H 7370 3796 50  0000 L CNN
-F 1 "120R" H 7370 3705 50  0000 L CNN
-F 2 "" V 7230 3750 50  0001 C CNN
-F 3 "~" H 7300 3750 50  0001 C CNN
-	1    7300 3750
-	1    0    0    -1
+P 7500 3600
+F 0 "R2" H 7570 3646 50  0000 L CNN
+F 1 "120R" H 7570 3555 50  0000 L CNN
+F 2 "Resistor_SMD:R_0603_1608Metric" V 7430 3600 50  0001 C CNN
+F 3 "~" H 7500 3600 50  0001 C CNN
+	1    7500 3600
+	0    -1   -1   0
 $EndComp
 $Comp
 L Connector_Generic:Conn_01x02 J3
 U 1 1 5E8F7136
-P 7800 3600
-F 0 "J3" H 7880 3592 50  0000 L CNN
-F 1 "Conn_01x02" H 7880 3501 50  0000 L CNN
-F 2 "" H 7800 3600 50  0001 C CNN
-F 3 "~" H 7800 3600 50  0001 C CNN
-	1    7800 3600
+P 8000 3800
+F 0 "J3" H 8080 3792 50  0000 L CNN
+F 1 "Conn_01x02" H 8080 3701 50  0000 L CNN
+F 2 "" H 8000 3800 50  0001 C CNN
+F 3 "~" H 8000 3800 50  0001 C CNN
+	1    8000 3800
 	1    0    0    -1
 $EndComp
@@
 P 4150 4450
 F 0 "X1" V 4104 4581 50  0000 L CNN
-F 1 "Crystal" V 4195 4581 50  0000 L CNN
-F 2 "" H 4150 4450 50  0001 C CNN
+F 1 "C115962" V 4195 4581 50  0000 L CNN
+F 2 "Crystal:Crystal_SMD_5032-2Pin_5.0x3.2mm" H 4150 4450 50  0001 C CNN
 F 3 "~" H 4150 4450 50  0001 C CNN
 	1    4150 4450
@@
 	-1   0    0    1
 $EndComp
+Wire Wire Line
+	7100 3900 7350 3900
+$Comp
+L Jumper:SolderJumper_2_Open JP?
+U 1 1 5EA60D30
+P 7350 3750
+F 0 "JP?" V 7304 3818 50  0000 L CNN
+F 1 "SolderJumper_2_Open" V 7395 3818 50  0000 L CNN
+F 2 "" H 7350 3750 50  0001 C CNN
+F 3 "~" H 7350 3750 50  0001 C CNN
+	1    7350 3750
+	0    1    1    0
+$EndComp
+Connection ~ 7350 3900
+Wire Wire Line
+	7350 3900 7800 3900
+Wire Wire Line
+	7150 3300 7800 3300
+Wire Wire Line
+	7800 3300 7800 3600
+Wire Wire Line
+	7150 3300 7150 3700
+Wire Wire Line
+	7650 3600 7800 3600
+Connection ~ 7800 3600
+Wire Wire Line
+	7800 3600 7800 3800
+Connection ~ 7350 4850
+Connection ~ 6900 4850
+Connection ~ 7350 4550
+Wire Wire Line
+	7350 4550 7550 4550
+Wire Wire Line
+	7350 4850 7850 4850
+Wire Wire Line
+	7000 4550 7350 4550
+Wire Wire Line
+	6250 4550 6900 4550
+Wire Wire Line
+	6250 4850 6900 4850
+Connection ~ 7000 4550
+Connection ~ 6900 4550
+Wire Wire Line
+	6900 4550 7000 4550
+Connection ~ 7150 4850
+Wire Wire Line
+	7150 4850 7350 4850
+Wire Wire Line
+	6900 4850 7150 4850
 $EndSCHEMATC

Commit message: Updated, added Capacitors
Parts:
- removed POW: LED, LED_SMD:LED_0603_1608Metric, symbol Device:LED
- removed R1: 1k, Resistor_SMD:R_0603_1608Metric, symbol Device:R
- C1: value 10uF/16V -> C7171; footprint (none) -> Resistor_SMD:R_1206_3216Metric
- J3: footprint (none) -> Connector_PinHeader_2.54mm:PinHeader_1x02_P2.54mm_Vertical
- J4: value Conn_01x06 -> Conn_01x07; footprint (none) -> Connector_PinHeader_2.54mm:PinHeader_1x07_P2.54mm_Vertical
- JP1: renamed from JP?; footprint (none) -> Jumper:SolderJumper-2_P1.3mm_Open_Pad1.0x1.5mm
Changed lines of the file:
@@
 	4000 3700 4300 3700
-$Comp
-L Device:R R1
-U 1 1 5E9187AF
-P 7700 4550
-F 0 "R1" V 7493 4550 50  0000 C CNN
-F 1 "1k" V 7584 4550 50  0000 C CNN
-F 2 "Resistor_SMD:R_0603_1608Metric" V 7630 4550 50  0001 C CNN
-F 3 "~" H 7700 4550 50  0001 C CNN
-	1    7700 4550
-	0    1    1    0
-$EndComp
 $Comp
 L power:GND #PWR?
@@
 	1    7150 4850
 	1    0    0    -1
-$EndComp
-$Comp
-L Device:LED POW
-U 1 1 5E91395F
-P 7850 4700
-F 0 "POW" V 7889 4583 50  0000 R CNN
-F 1 "LED" V 7798 4583 50  0000 R CNN
-F 2 "LED_SMD:LED_0603_1608Metric" H 7850 4700 50  0001 C CNN
-F 3 "~" H 7850 4700 50  0001 C CNN
-	1    7850 4700
-	0    -1   -1   0
 $EndComp
 $Comp
@@
 P 6250 4700
 F 0 "C1" H 6368 4746 50  0000 L CNN
-F 1 "10uF/16V" H 6368 4655 50  0000 L CNN
-F 2 "" H 6288 4550 50  0001 C CNN
+F 1 "C7171" H 6368 4655 50  0000 L CNN
+F 2 "Resistor_SMD:R_1206_3216Metric" H 6288 4550 50  0001 C CNN
 F 3 "~" H 6250 4700 50  0001 C CNN
 	1    6250 4700
@@
 F 0 "J3" H 8080 3792 50  0000 L CNN
 F 1 "Conn_01x02" H 8080 3701 50  0000 L CNN
-F 2 "" H 8000 3800 50  0001 C CNN
+F 2 "Connector_PinHeader_2.54mm:PinHeader_1x02_P2.54mm_Vertical" H 8000 3800 50  0001 C CNN
 F 3 "~" H 8000 3800 50  0001 C CNN
 	1    8000 3800
@@
 P 3800 3600
 F 0 "J4" H 3718 3075 50  0000 C CNN
-F 1 "Conn_01x06" H 3718 3166 50  0000 C CNN
-F 2 "" H 3800 3600 50  0001 C CNN
+F 1 "Conn_01x07" H 3718 3166 50  0000 C CNN
+F 2 "Connector_PinHeader_2.54mm:PinHeader_1x07_P2.54mm_Vertical" H 3800 3600 50  0001 C CNN
 F 3 "~" H 3800 3600 50  0001 C CNN
 	1    3800 3600
@@
 	7100 3900 7350 3900
 $Comp
-L Jumper:SolderJumper_2_Open JP?
+L Jumper:SolderJumper_2_Open JP1
 U 1 1 5EA60D30
 P 7350 3750
-F 0 "JP?" V 7304 3818 50  0000 L CNN
+F 0 "JP1" V 7304 3818 50  0000 L CNN
 F 1 "SolderJumper_2_Open" V 7395 3818 50  0000 L CNN
-F 2 "" H 7350 3750 50  0001 C CNN
+F 2 "Jumper:SolderJumper-2_P1.3mm_Open_Pad1.0x1.5mm" H 7350 3750 50  0001 C CNN
 F 3 "~" H 7350 3750 50  0001 C CNN
 	1    7350 3750
@@
 Wire Wire Line
 	7800 3600 7800 3800
-Connection ~ 7350 4850
 Connection ~ 6900 4850
-Connection ~ 7350 4550
-Wire Wire Line
-	7350 4550 7550 4550
-Wire Wire Line
-	7350 4850 7850 4850
 Wire Wire Line
 	7000 4550 7350 4550
